File: pcb/Dragtser_PCB/Dragtser_PCB.kicad_sch (KiCad schematic)
At the start: 0 parts

Commit message: esquemático pcb com atribuição de footprits
Parts:
- added J1, J2: Conn_01x09_Pin, Connector_PinHeader_2.54mm:PinHeader_1x09_P2.54mm_Vertical, symbol Connector:Conn_01x09_Pin
- added J10, J11, J7, J8, J9: Conn_01x02_Pin, TerminalBlock_Phoenix:TerminalBlock_Phoenix_MKDS-1,5-2-5.08_1x02_P5.08mm_Horizontal, symbol Connector:Conn_01x02_Pin
- added J12, J13: Conn_01x05_Pin, Connector_PinHeader_2.54mm:PinHeader_1x05_P2.54mm_Vertical, symbol Connector:Conn_01x05_Pin
- added J3, J4, J5: Conn_01x04_Pin, Connector_PinHeader_2.54mm:PinHeader_1x04_P2.54mm_Vertical, symbol Connector:Conn_01x04_Pin
- added J6: Conn_01x02_Pin, Connector_AMASS:AMASS_XT30U-M_1x02_P5.0mm_Vertical, symbol Connector:Conn_01x02_Pin
Connections:
- new net 3.3V: J1.3 (Pin_3), J3.1 (Pin_1), J4.1 (Pin_1), J5.1 (Pin_1)
- new net 5V: J1.1 (Pin_1), J12.1 (Pin_1), J13.1 (Pin_1)
- new net DIR+: J10.1 (Pin_1), J8.1 (Pin_1)
- new net DIR-: J10.2 (Pin_2), J8.2 (Pin_2)
- new net ESQ+: J11.1 (Pin_1), J9.1 (Pin_1)
- new net ESQ-: J11.2 (Pin_2), J9.2 (Pin_2)
- new net GND: J1.2 (Pin_2), J12.5 (Pin_5), J13.5 (Pin_5), J3.2 (Pin_2), J4.2 (Pin_2), J5.2 (Pin_2), J6.2 (Pin_2), J7.2 (Pin_2)
- new net GP1: J1.4 (Pin_4), J3.3 (Pin_3), J4.3 (Pin_3)
- new net GP10: J2.6 (Pin_6)
- new net GP11: J2.5 (Pin_5)
- new net GP12: J2.4 (Pin_4)
- new net GP13: J2.3 (Pin_3)
- new net GP2: J1.5 (Pin_5), J3.4 (Pin_4), J4.4 (Pin_4)
- new net GP3: J1.6 (Pin_6), J5.3 (Pin_3)
- new net GP4: J1.7 (Pin_7), J12.2 (Pin_2)
- new net GP5: J1.8 (Pin_8), J12.3 (Pin_3)
- new net GP6: J1.9 (Pin_9), J12.4 (Pin_4)
- new net GP7: J13.3 (Pin_3), J2.9 (Pin_9)
- new net GP8: J13.4 (Pin_4), J2.8 (Pin_8)
- new net GP9: J2.7 (Pin_7)
- new net RX: J2.2 (Pin_2)
- new net TX: J2.1 (Pin_1)
- new net VCC_BATERIA: J6.1 (Pin_1), J7.1 (Pin_1)
- no-connect marks 0 -> 2
